File: pcbs/motorTesting Rig/controlmodule-ra.sch (EAGLE design)
At the start: 31 parts, among them Q1 16mhz, U1 ATMEGA328P_TQFP

Commit message: control board v1.3, moved stuff to bottom side to avoid aluminum shavings
Parts:
- added C10: 10u, rcl:C-EUC0805
- added C9: 1u, rcl:C-EUC0805
Connections:
- net XTAL1 renamed XTAL_P
- net XTAL2 renamed XTAL_N
- net GND: now also C10.1, C9.1
- net VCC: now also C10.2, C9.2
Changed lines of the file:
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@@
 <part name="GND13" library="supply1" library_urn="urn:adsk.eagle:library:371" deviceset="GND" device=""/>
 <part name="GND14" library="supply1" library_urn="urn:adsk.eagle:library:371" deviceset="GND" device=""/>
+<part name="P+9" library="supply1" library_urn="urn:adsk.eagle:library:371" deviceset="VCC" device=""/>
+<part name="C9" library="rcl" library_urn="urn:adsk.eagle:library:334" deviceset="C-EU" device="C0805" package3d_urn="urn:adsk.eagle:package:23617/2" value="1u"/>
+<part name="C10" library="rcl" library_urn="urn:adsk.eagle:library:334" deviceset="C-EU" device="C0805" package3d_urn="urn:adsk.eagle:package:23617/2" value="10u"/>
+<part name="GND15" library="supply1" library_urn="urn:adsk.eagle:library:371" deviceset="GND" device=""/>
 </parts>
 <sheets>
@@
 <attribute name="VALUE" x="208.28" y="121.92" size="1.778" layer="96"/>
 </instance>
+<instance part="P+9" gate="VCC" x="114.3" y="35.56" smashed="yes">
+<attribute name="VALUE" x="116.84" y="38.1" size="1.778" layer="96" rot="R180"/>
+</instance>
+<instance part="C9" gate="G$1" x="109.22" y="22.86" smashed="yes" rot="R180">
+<attribute name="NAME" x="107.696" y="22.479" size="1.778" layer="95" rot="R180"/>
+<attribute name="VALUE" x="107.696" y="27.559" size="1.778" layer="96" rot="R180"/>
+</instance>
+<instance part="C10" gate="G$1" x="119.38" y="22.86" smashed="yes" rot="R180">
+<attribute name="NAME" x="117.856" y="22.479" size="1.778" layer="95" rot="R180"/>
+<attribute name="VALUE" x="117.856" y="27.559" size="1.778" layer="96" rot="R180"/>
+</instance>
+<instance part="GND15" gate="1" x="114.3" y="12.7" smashed="yes">
+<attribute name="VALUE" x="111.76" y="10.16" size="1.778" layer="96"/>
+</instance>
 </instances>
 <busses>
 </busses>
 <nets>
-<net name="XTAL2" class="0">
+<net name="XTAL_N" class="0">
 <segment>
 <pinref part="Q1" gate="G$1" pin="1"/>
@@
 <wire x1="111.76" y1="119.38" x2="104.14" y2="119.38" width="0.1524" layer="91"/>
 <junction x="104.14" y="119.38"/>
+<label x="104.14" y="116.84" size="1.778" layer="95"/>
 </segment>
 </net>
-<net name="XTAL1" class="0">
+<net name="XTAL_P" class="0">
 <segment>
 <pinref part="C1" gate="G$1" pin="2"/>
@@
 <wire x1="104.14" y1="124.46" x2="111.76" y2="124.46" width="0.1524" layer="91"/>
 <junction x="104.14" y="124.46"/>
+<label x="104.14" y="124.46" size="1.778" layer="95"/>
 </segment>
 </net>
@@
 <wire x1="210.82" y1="129.54" x2="210.82" y2="127" width="0.1524" layer="91"/>
 </segment>
+<segment>
+<pinref part="C9" gate="G$1" pin="1"/>
+<wire x1="109.22" y1="20.32" x2="109.22" y2="17.78" width="0.1524" layer="91"/>
+<wire x1="109.22" y1="17.78" x2="114.3" y2="17.78" width="0.1524" layer="91"/>
+<wire x1="114.3" y1="17.78" x2="119.38" y2="17.78" width="0.1524" layer="91"/>
+<wire x1="119.38" y1="17.78" x2="119.38" y2="20.32" width="0.1524" layer="91"/>
+<pinref part="GND15" gate="1" pin="GND"/>
+<wire x1="114.3" y1="15.24" x2="114.3" y2="17.78" width="0.1524" layer="91"/>
+<junction x="114.3" y="17.78"/>
+<pinref part="C10" gate="G$1" pin="1"/>
+</segment>
 </net>
 <net name="VCC" class="0">
@@
 <pinref part="P+11" gate="VCC" pin="VCC"/>
 </segment>
+<segment>
+<pinref part="C9" gate="G$1" pin="2"/>
+<wire x1="109.22" y1="27.94" x2="109.22" y2="30.48" width="0.1524" layer="91"/>
+<wire x1="109.22" y1="30.48" x2="114.3" y2="30.48" width="0.1524" layer="91"/>
+<wire x1="114.3" y1="30.48" x2="119.38" y2="30.48" width="0.1524" layer="91"/>
+<wire x1="119.38" y1="30.48" x2="119.38" y2="27.94" width="0.1524" layer="91"/>
+<pinref part="P+9" gate="VCC" pin="VCC"/>
+<wire x1="114.3" y1="30.48" x2="114.3" y2="33.02" width="0.1524" layer="91"/>
+<junction x="114.3" y="30.48"/>
+<pinref part="C10" gate="G$1" pin="2"/>
+</segment>
 </net>
